Commit message: ROS 包名改为 PM01_Marathon。

File: urdf/pm01_edu.urdf (robot description, URDF)
Before this commit: robot pm01_edu, 37 links, 36 joints
Links:
- link LINK_ANKLE_PITCH_L: geometry visual mesh filename=package://PM01_Marathon/meshes/LINK_ANKLE_PITCH_L.dae
- link LINK_ANKLE_PITCH_R: geometry visual mesh filename=package://PM01_Marathon/meshes/LINK_ANKLE_PITCH_R.dae
- link LINK_ANKLE_ROLL_L: geometry visual mesh filename=package://PM01_Marathon/meshes/LINK_ANKLE_ROLL_L.dae
- link LINK_ANKLE_ROLL_R: geometry visual mesh filename=package://PM01_Marathon/meshes/LINK_ANKLE_ROLL_R.dae
- link LINK_BASE: geometry visual mesh filename=package://PM01_Marathon/meshes/LINK_BASE.dae
- link LINK_ELBOW_PITCH_L: geometry visual mesh filename=package://PM01_Marathon/meshes/LINK_ELBOW_PITCH_L.dae
- link LINK_ELBOW_PITCH_R: geometry visual mesh filename=package://PM01_Marathon/meshes/LINK_ELBOW_PITCH_R.dae
- link LINK_ELBOW_YAW_L: geometry visual mesh filename=package://PM01_Marathon/meshes/LINK_ELBOW_YAW_L.dae
- link LINK_ELBOW_YAW_R: geometry visual mesh filename=package://PM01_Marathon/meshes/LINK_ELBOW_YAW_R.dae
- link LINK_HEAD_YAW: geometry visual mesh filename=package://PM01_Marathon/meshes/LINK_HEAD_YAW.dae
- link LINK_HIP_PITCH_L: geometry visual mesh filename=package://PM01_Marathon/meshes/LINK_HIP_PITCH_L.dae
- link LINK_HIP_PITCH_R: geometry visual mesh filename=package://PM01_Marathon/meshes/LINK_HIP_PITCH_R.dae
- link LINK_HIP_ROLL_L: geometry visual mesh filename=package://PM01_Marathon/meshes/LINK_HIP_ROLL_L.dae
- link LINK_HIP_ROLL_R: geometry visual mesh filename=package://PM01_Marathon/meshes/LINK_HIP_ROLL_R.dae
- link LINK_HIP_YAW_L: geometry visual mesh filename=package://PM01_Marathon/meshes/LINK_HIP_YAW_L.dae
- link LINK_HIP_YAW_R: geometry visual mesh filename=package://PM01_Marathon/meshes/LINK_HIP_YAW_R.dae
- link LINK_KNEE_PITCH_L: geometry visual mesh filename=package://PM01_Marathon/meshes/LINK_KNEE_PITCH_L.dae
- link LINK_KNEE_PITCH_R: geometry visual mesh filename=package://PM01_Marathon/meshes/LINK_KNEE_PITCH_R.dae
- link LINK_SHOULDER_PITCH_L: geometry visual mesh filename=package://PM01_Marathon/meshes/LINK_SHOULDER_PITCH_L.dae
- link LINK_SHOULDER_PITCH_R: geometry visual mesh filename=package://PM01_Marathon/meshes/LINK_SHOULDER_PITCH_R.dae
- link LINK_SHOULDER_ROLL_L: geometry visual mesh filename=package://PM01_Marathon/meshes/LINK_SHOULDER_ROLL_L.dae
- link LINK_SHOULDER_ROLL_R: geometry visual mesh filename=package://PM01_Marathon/meshes/LINK_SHOULDER_ROLL_R.dae
- link LINK_SHOULDER_YAW_L: geometry visual mesh filename=package://PM01_Marathon/meshes/LINK_SHOULDER_YAW_L.dae
- link LINK_SHOULDER_YAW_R: geometry visual mesh filename=package://PM01_Marathon/meshes/LINK_SHOULDER_YAW_R.dae
- link LINK_TORSO_YAW: geometry visual mesh filename=package://PM01_Marathon/meshes/LINK_TORSO_YAW.dae

Commit message: ROS 包名改为 pm01_marathon。

File: urdf/pm01_edu.urdf (robot description, URDF)
Before this commit: robot pm01_edu, 37 links, 36 joints
Links:
- link LINK_ANKLE_PITCH_L: geometry visual mesh filename=package://pm01_marathon/meshes/LINK_ANKLE_PITCH_L.dae
- link LINK_ANKLE_PITCH_R: geometry visual mesh filename=package://pm01_marathon/meshes/LINK_ANKLE_PITCH_R.dae
- link LINK_ANKLE_ROLL_L: geometry visual mesh filename=package://pm01_marathon/meshes/LINK_ANKLE_ROLL_L.dae
- link LINK_ANKLE_ROLL_R: geometry visual mesh filename=package://pm01_marathon/meshes/LINK_ANKLE_ROLL_R.dae
- link LINK_BASE: geometry visual mesh filename=package://pm01_marathon/meshes/LINK_BASE.dae
- link LINK_ELBOW_PITCH_L: geometry visual mesh filename=package://pm01_marathon/meshes/LINK_ELBOW_PITCH_L.dae
- link LINK_ELBOW_PITCH_R: geometry visual mesh filename=package://pm01_marathon/meshes/LINK_ELBOW_PITCH_R.dae
- link LINK_ELBOW_YAW_L: geometry visual mesh filename=package://pm01_marathon/meshes/LINK_ELBOW_YAW_L.dae
- link LINK_ELBOW_YAW_R: geometry visual mesh filename=package://pm01_marathon/meshes/LINK_ELBOW_YAW_R.dae
- link LINK_HEAD_YAW: geometry visual mesh filename=package://pm01_marathon/meshes/LINK_HEAD_YAW.dae
- link LINK_HIP_PITCH_L: geometry visual mesh filename=package://pm01_marathon/meshes/LINK_HIP_PITCH_L.dae
- link LINK_HIP_PITCH_R: geometry visual mesh filename=package://pm01_marathon/meshes/LINK_HIP_PITCH_R.dae
- link LINK_HIP_ROLL_L: geometry visual mesh filename=package://pm01_marathon/meshes/LINK_HIP_ROLL_L.dae
- link LINK_HIP_ROLL_R: geometry visual mesh filename=package://pm01_marathon/meshes/LINK_HIP_ROLL_R.dae
- link LINK_HIP_YAW_L: geometry visual mesh filename=package://pm01_marathon/meshes/LINK_HIP_YAW_L.dae
- link LINK_HIP_YAW_R: geometry visual mesh filename=package://pm01_marathon/meshes/LINK_HIP_YAW_R.dae
- link LINK_KNEE_PITCH_L: geometry visual mesh filename=package://pm01_marathon/meshes/LINK_KNEE_PITCH_L.dae
- link LINK_KNEE_PITCH_R: geometry visual mesh filename=package://pm01_marathon/meshes/LINK_KNEE_PITCH_R.dae
- link LINK_SHOULDER_PITCH_L: geometry visual mesh filename=package://pm01_marathon/meshes/LINK_SHOULDER_PITCH_L.dae
- link LINK_SHOULDER_PITCH_R: geometry visual mesh filename=package://pm01_marathon/meshes/LINK_SHOULDER_PITCH_R.dae
- link LINK_SHOULDER_ROLL_L: geometry visual mesh filename=package://pm01_marathon/meshes/LINK_SHOULDER_ROLL_L.dae
- link LINK_SHOULDER_ROLL_R: geometry visual mesh filename=package://pm01_marathon/meshes/LINK_SHOULDER_ROLL_R.dae
- link LINK_SHOULDER_YAW_L: geometry visual mesh filename=package://pm01_marathon/meshes/LINK_SHOULDER_YAW_L.dae
- link LINK_SHOULDER_YAW_R: geometry visual mesh filename=package://pm01_marathon/meshes/LINK_SHOULDER_YAW_R.dae
- link LINK_TORSO_YAW: geometry visual mesh filename=package://pm01_marathon/meshes/LINK_TORSO_YAW.dae

Commit message: 用 zqsa01 策略给出腿部姿态，并等控制器起来再打开 Gazebo 窗口。

File: urdf/pm01_edu.urdf (robot description, URDF)
Before this commit: robot pm01_edu, 37 links, 36 joints
Joints:
- joint J00_HIP_PITCH_L: axis (none) -> 0 0.96593 -0.25882; limit (none) -> lower=-3.141 upper=2.443 effort=2 velocity=8; type fixed -> revolute
- joint J01_HIP_ROLL_L: axis (none) -> 1 0 0; limit (none) -> lower=-0.436 upper=2.094 effort=2 velocity=8; type fixed -> revolute
- joint J02_HIP_YAW_L: axis (none) -> 0 0 1; limit (none) -> lower=-1.57 upper=4.014 effort=2 velocity=8; type fixed -> revolute
- joint J03_KNEE_PITCH_L: axis (none) -> 0 1 0; limit (none) -> lower=-0.3491 upper=2.3911 effort=2 velocity=8; type fixed -> revolute
- joint J04_ANKLE_PITCH_L: axis (none) -> 0 1 0; limit (none) -> lower=-0.6807 upper=0.7243 effort=2 velocity=8; type fixed -> revolute
- joint J05_ANKLE_ROLL_L: axis (none) -> 1 0 0; limit (none) -> lower=-0.2618 upper=0.2618 effort=2 velocity=8; type fixed -> revolute
- joint J06_HIP_PITCH_R: axis (none) -> 0 0.96593 0.25882; limit (none) -> lower=-3.141 upper=2.443 effort=2 velocity=8; type fixed -> revolute
- joint J07_HIP_ROLL_R: axis (none) -> 1 0 0; limit (none) -> lower=-2.094 upper=0.436 effort=2 velocity=8; type fixed -> revolute
- joint J08_HIP_YAW_R: axis (none) -> 0 0 1; limit (none) -> lower=-4.014 upper=1.57 effort=2 velocity=8; type fixed -> revolute
- joint J09_KNEE_PITCH_R: axis (none) -> 0 1 0; limit (none) -> lower=-0.3491 upper=2.3911 effort=2 velocity=8; type fixed -> revolute
- joint J10_ANKLE_PITCH_R: axis (none) -> 0 1 0; limit (none) -> lower=-0.6807 upper=0.7243 effort=2 velocity=8; type fixed -> revolute
- joint J11_ANKLE_ROLL_R: axis (none) -> 1 0 0; limit (none) -> lower=-0.2618 upper=0.2618 effort=2 velocity=8; type fixed -> revolute
